Commit message: Faz 0 ve Faz 1: ROS 2 robot altyapısı ve komut merkezi eklendi

File: src/robot_description/urdf/robot.urdf (robot description, URDF)
Before this commit: robot six_axis_robot, 3 links, 2 joints
Links:
- added link link_3; visual box size=0.05 0.05 0.3
- added link link_4; visual cylinder length=0.2 radius=0.04
- added link link_5; visual box size=0.04 0.04 0.15
- added link link_6; visual cylinder length=0.05 radius=0.03
- link base_link: geometry visual cylinder length=0.08 radius=0.12
- link link_2: geometry visual box size=0.06 0.06 0.35
Joints:
- added joint joint_3: type revolute, parent link_2, child link_3, origin xyz=0 0 0.35, axis 0 1 0, limit lower=-2.0 upper=2.0 effort=100 velocity=1.0
- added joint joint_4: type revolute, parent link_3, child link_4, origin xyz=0 0 0.3, axis 0 0 1, limit lower=-3.14 upper=3.14 effort=100 velocity=1.0
- added joint joint_5: type revolute, parent link_4, child link_5, origin xyz=0 0 0.2, axis 0 1 0, limit lower=-1.57 upper=1.57 effort=100 velocity=1.0
- added joint joint_6: type revolute, parent link_5, child link_6, origin xyz=0 0 0.15, axis 0 0 1, limit lower=-3.14 upper=3.14 effort=100 velocity=1.0
- joint joint_1: origin xyz=0 0 0.05 -> xyz=0 0 0.04
