Commit message: Fix robot model config: collision geometry, ACM, joint limits
- URDF: add <collision> and placeholder <inertial> to all links (without collision
  geometry MoveIt ignored planning-scene obstacles)
- SRDF: disable collisions for adjacent links, add cnc/pc/dik group states
- joint_limits.yaml: merge duplicated top-level key, enable accel limits
- remove dead robot.srdf (never loaded, conflicting robot name)
- robot_description: install() before ament_package()

Co-Authored-By: Claude Sonnet 5.5 <noreply@anthropic.com>
Claude-Session: https://claude.ai/code/session_01QReM5HVwMn8fE3qZwBmP7V

File: src/robot_description/urdf/robot.urdf (robot description, URDF)
Before this commit: robot six_axis_robot, 7 links, 6 joints
Links:
- link base_link: geometry collision cylinder length=0.08 radius=0.12; visual cylinder length=0.08 radius=0.12
- link link_1: mass None -> 2.0; geometry collision cylinder length=0.2 radius=0.08; visual cylinder length=0.2 radius=0.08
- link link_2: mass None -> 1.5; geometry collision box size=0.06 0.06 0.35; visual box size=0.06 0.06 0.35
- link link_3: mass None -> 1.0; geometry collision box size=0.05 0.05 0.3; visual box size=0.05 0.05 0.3
- link link_4: mass None -> 0.6; geometry collision cylinder length=0.2 radius=0.04; visual cylinder length=0.2 radius=0.04
- link link_5: mass None -> 0.4; geometry collision box size=0.04 0.04 0.15; visual box size=0.04 0.04 0.15
- link link_6: mass None -> 0.2; geometry collision cylinder length=0.05 radius=0.03; visual cylinder length=0.05 radius=0.03

Commit message: Add Gazebo physics mode (gz_ros2_control), keep mock mode as default
- xacro: use_gazebo arg swaps mock_components for gz_ros2_control/GazeboSimSystem;
  massless world link + masa joint in both modes (matches the SRDF virtual joint)
- robot.urdf: base_link gets a placeholder <inertial> (without it sdformat lumps the link
  into the world and joint_1 loses its parent)
- gazebo.launch.py: headless gz server, /clock bridge, spawn, controller spawners,
  move_group on sim time (headless:=false for the GUI)
- run_selftest.sh takes mock|gazebo; CI and compose run both
- verified locally: 7/7 on mock and on Gazebo, 4 extra Gazebo runs, sim time ~0.93x real

Co-Authored-By: Claude Sonnet 5.5 <noreply@anthropic.com>
Claude-Session: https://claude.ai/code/session_01QReM5HVwMn8fE3qZwBmP7V

File: src/robot_description/urdf/robot.urdf (robot description, URDF)
Before this commit: robot six_axis_robot, 7 links, 6 joints
Links:
- link base_link: mass None -> 5.0

File: src/robot_moveit_config/config/six_axis_robot.ros2_control.xacro (robot description, xacro)
@@ -1,10 +1,16 @@
 <?xml version="1.0"?>
 <robot xmlns:xacro="http://www.ros.org/wiki/xacro">
-    <xacro:macro name="six_axis_robot_ros2_control" params="name initial_positions_file">
+    <xacro:macro name="six_axis_robot_ros2_control" params="name initial_positions_file use_gazebo:=false">
         <xacro:property name="initial_positions" value="${xacro.load_yaml(initial_positions_file)['initial_positions']}"/>
         <ros2_control name="${name}" type="system">
             <hardware>
-                <!-- By default, set up controllers for simulation. This won't work on real hardware -->
-                <plugin>mock_components/GenericSystem</plugin>
+                <!-- Default: mock hardware (no physics). use_gazebo:=true: Gazebo physics. Neither works
+                     on real hardware. -->
+                <xacro:if value="${use_gazebo}">
+                    <plugin>gz_ros2_control/GazeboSimSystem</plugin>
+                </xacro:if>
+                <xacro:unless value="${use_gazebo}">
+                    <plugin>mock_components/GenericSystem</plugin>
+                </xacro:unless>
             </hardware>
             <joint name="joint_1">

File: src/robot_moveit_config/config/six_axis_robot.urdf.xacro (robot description, xacro)
@@ -2,8 +2,28 @@
 <robot xmlns:xacro="http://www.ros.org/wiki/xacro" name="six_axis_robot">
     <xacro:arg name="initial_positions_file" default="initial_positions.yaml" />
+    <!-- false: mock_components (no physics, default). true: Gazebo physics via gz_ros2_control. -->
+    <xacro:arg name="use_gazebo" default="false" />
     <!-- Import six_axis_robot urdf file -->
     <xacro:include filename="$(find robot_description)/urdf/robot.urdf" />
     <!-- Import control_xacro -->
     <xacro:include filename="six_axis_robot.ros2_control.xacro" />
-    <xacro:six_axis_robot_ros2_control name="FakeSystem" initial_positions_file="$(arg initial_positions_file)"/>
+    <xacro:six_axis_robot_ros2_control name="FakeSystem"
+                                       initial_positions_file="$(arg initial_positions_file)"
+                                       use_gazebo="$(arg use_gazebo)"/>
+    <!-- base_link is fixed to the world in both modes (same joint name as the SRDF virtual joint).
+         Gazebo needs it, otherwise the arm falls over; it also keeps `world` (massless) as the
+         kinematic root, so KDL never sees an inertia on the root link. -->
+    <link name="world"/>
+    <joint name="masa" type="fixed">
+        <parent link="world"/>
+        <child link="base_link"/>
+    </joint>
+    <xacro:if value="$(arg use_gazebo)">
+        <gazebo>
+            <plugin filename="gz_ros2_control-system"
+                    name="gz_ros2_control::GazeboSimROS2ControlPlugin">
+                <parameters>$(find robot_moveit_config)/config/ros2_controllers.yaml</parameters>
+            </plugin>
+        </gazebo>
+    </xacro:if>
 </robot>
